File: board/hw-TS1B.kicad_pcb (KiCad board)
At the start: 2 copper layers, 38 x 16 mm, 22 parts, among them J1 3V3, J2 Conn_01x02, U1 STM32L011D3Px, U2 CMT2110A, X1 SWD, X2 SG-210STF

Commit message: WIP
Parts:
- added C9: 100n, Capacitor_SMD:C_0805_2012Metric, F.Cu at (163.0, 73.0)
- U1: value STM32L011D3Px -> STM32L031F6Px; footprint Package_SO:TSSOP-14_4.4x5mm_P0.65mm -> Package_SO:TSSOP-20_4.4x6.5mm_P0.65mm
- moved D1 2.50 mm to (187.0, 77.0), turned to 180 degrees
- moved R2 2.50 mm to (187.0, 79.5), turned to 0 degrees
- moved C6 1.90 mm to (170.8, 79.8), turned to 180 degrees
- moved U1 1.00 mm to (170.0, 73.5)
- moved C3 0.06 mm to (163.0, 70.8)
Connections:
- D1 pad 1: GND -> Net-(D1-Pad1)
- D1 pad 2: Net-(D1-Pad2) -> /LED
- R2 pad 1: Net-(D1-Pad2) -> GND
- R2 pad 2: /LED -> Net-(D1-Pad1)
- U1 pad 1: Net-(U1-Pad1) -> GND
- U1 pad 10: VDD -> /TEMP_PWR
- U1 pad 12: /TEMP_PWR -> /RF_DATA
- U1 pad 13: /SWDIO -> /RF_CLK
- U1 pad 14: /SWCLK -> (no net)
- U1 pad 2: /RF_DATA -> (no net)
- U1 pad 3: /RF_CLK -> (no net)
- U1 pad 5: /26MHZ -> VDD
- U1 pad 6: /OSC_EN -> /26MHZ
- U1 pad 7: /LED -> /OSC_EN
- U1 pad 8: /TEMP_SNS -> /LED
- U1 pad 9: GND -> /TEMP_SNS
Routing:
- net /TEMP_SNS: track 15.0 -> 21.4 mm, vias 0 -> 2
- net /OSC_EN: track 11.6 -> 16.9 mm, vias 0 -> 2
- net /RF_DATA: track 18.6 -> 14.4 mm
- net VDD: track 61.3 -> 64.7 mm
- net GND: track 21.0 -> 23.8 mm, vias 9 -> 10
- net /TEMP_PWR: track 15.1 -> 17.9 mm, vias 0 -> 2
- net Net-(D1-Pad2): track 2.50 -> 0.00 mm
- net Net-(D1-Pad1): track 0.00 -> 2.50 mm
- net /26MHZ: track 17.6 -> 16.3 mm
- net /LED: track 23.7 -> 22.9 mm
- net /RF_CLK: track 15.6 -> 15.4 mm, vias 0 -> 2
Other:
- board text added: "TS1B v1.1"
- board text removed: "TS1B v1.0"

Commit message: WIP
Parts:
- removed C2: 100n, Capacitor_SMD:C_0805_2012Metric
- U1: value STM32L031F6Px -> ATSAMD11C14A-SS; footprint Package_SO:TSSOP-20_4.4x6.5mm_P0.65mm -> Package_SO:SOIC-14_3.9x8.7mm_P1.27mm
- moved C6 5.57 mm to (166.4, 83.2)
- moved U2 2.41 mm to (170.2, 80.6), turned to 270 degrees
- moved U1 2.09 mm to (172.1, 73.7), turned to 90 degrees
- moved L1 1.27 mm to (175.3, 79.4), turned to 0 degrees
- moved C5 0.29 mm to (165.7, 79.4), turned to 180 degrees
Connections:
- U1 pad 1: GND -> /TEMP_SNS
- U1 pad 10: /TEMP_PWR -> Net-(U1-Pad10)
- U1 pad 11: /TEMP_PWR -> GND
- U1 pad 12: /RF_DATA -> VDD
- U1 pad 13: /RF_CLK -> /TEMP_PWR
- U1 pad 14: (no net) -> /TEMP_PWR
- U1 pad 2: (no net) -> /26MHZ
- U1 pad 3: (no net) -> /OSC_EN
- U1 pad 4: Net-(C3-Pad1) -> /RF_DATA
- U1 pad 5: VDD -> /RF_CLK
- U1 pad 6: /26MHZ -> Net-(C3-Pad1)
- U1 pad 7: /OSC_EN -> /SWCLK
- U1 pad 8: /LED -> /SWDIO
- U1 pad 9: /TEMP_SNS -> /LED
Routing:
- net Net-(C3-Pad1): track 3.85 -> 13.4 mm, vias 0 -> 3
- net /RF_DATA: track 14.4 -> 4.94 mm, vias 2 -> 0
- net /LED: track 22.9 -> 15.9 mm
- net /RF_CLK: track 15.4 -> 8.94 mm, vias 2 -> 0
- net /TEMP_PWR: track 17.9 -> 23.9 mm
- net Net-(C1-Pad2): track 4.50 -> 9.84 mm
- net /SWDIO: track 9.67 -> 6.04 mm
- net /OSC_EN: track 16.9 -> 20.5 mm
- net GND: track 23.8 -> 27.3 mm, vias 10 -> 9
- net VDD: track 64.7 -> 61.3 mm, vias 3 -> 4
- net Net-(C5-Pad1): track 4.05 -> 7.35 mm, vias 0 -> 2
- net /26MHZ: track 16.3 -> 18.6 mm
Other:
- board text added: "TS1B v1.2"
- board text removed: "TS1B v1.1"
